File: CH572D-Board/CH572D-Board.kicad_pcb (KiCad board)
At the start: 2 copper layers, 13 parts, among them Y1 32mhz

Commit message: small work mostlty useless
Parts:
- added J1: Conn_USB_C_Socket, Footprint:Conn_USB_C_Socket_GCT_USB4125-GF-A-0190, F.Cu at (147.2, 128.0)
- added U2: TCR2EF33_LMCT, Footprint:voltage regulator, F.Cu at (144.1, 137.2)
- C5: value 10uF -> 2.2uF; footprint Personal:0603 -> Footprint:0603
- E1: footprint Personal:ceramic antenna -> Footprint:pcbantenna
- U1: footprint Ch572D:CH572D -> Footprint:CH572D
- Y1: footprint Personal:32mhz crystal -> Footprint:32mhz crystal
Connections:
- E1 pad 1: Net-(E1-Pad1) -> Net-(U1-ANT)
- U1 pad 5: ANTENNA -> Net-(U1-ANT)
