File: CH572D-Board/CH572D-Board.kicad_pcb (KiCad board)
At the start: 2 copper layers, 14 parts, among them J1 12402012E212A, U2 MIC5504-3.3YM5-TR, Y1 32mhz

Commit message: dont eve nknow
Parts:
- R1, R2: moved to B.Cu
- moved E1 19.2 mm to (104.6, 95.9), turned to 90 degrees
- moved U1 12.5 mm to (109.1, 86.0)
- moved U2 7.55 mm to (110.2, 94.3)
- moved R2 3.34 mm to (111.8, 84.8)
- moved Y1 3.04 mm to (110.5, 65.2)
- moved R1 1.67 mm to (111.7, 90.7)
- moved R3 0.65 mm to (117.1, 94.4)
- moved S1 0.65 mm to (116.5, 94.4)
Routing:
- net Net-(R3-Pad1): track 1.74 -> 0.00 mm

Commit message: some work
Parts:
- removed C4: 0.1uF, Personal:0603
- added C6: 2.2uF, Personal:0603, F.Cu at (158.6, 132.4)
- added C7: 0.1uF, Personal:0603, F.Cu at (155.4, 132.4)
- added J2: Conn_PinHeader_1x07_P2.54mm_Vertical_THT_D1mm, fab:PinHeader_1x07_P2.54mm_Vertical_THT_D1mm, F.Cu at (1.82, 1.82)
- added L1: 3.9nH, Personal:0603, F.Cu at (154.8, 118.8)
- C3: value 10uF -> 1.5pF
- C5: value 10uF -> 2.2uF
- E1: value ~ -> AMCA31-2R450G-S1F-T3; footprint Personal:antenna -> Personal:ceramic antenna
- R1, R2, R3: moved to F.Cu
- moved C2 100.9 mm to (159.0, 136.4), turned to 90 degrees
- moved C1 98.5 mm to (155.4, 133.8), turned to 180 degrees
- moved C5 93.2 mm to (158.5, 133.8), turned to 180 degrees
- moved Y1 85.1 mm to (164.5, 131.0), turned to 90 degrees
- moved C3 82.3 mm to (151.3, 120.7)
- moved U1 70.9 mm to (160.2, 135.1), turned to -90 degrees
- moved J1 70.3 mm to (160.2, 143.9), turned to 0 degrees
- moved R2 69.7 mm to (154.4, 139.8)
- moved S1 69.1 mm to (167.3, 141.3), turned to 90 degrees
- moved R1 67.6 mm to (154.4, 143.0)
- moved U2 62.2 mm to (156.1, 136.4)
- moved R3 61.6 mm to (161.3, 137.3), turned to 180 degrees
- moved E1 59.9 mm to (158.9, 121.1), turned to -90 degrees
Connections:
- net D+ renamed PA1
- net D- renamed PA0
- C3 pad 2: +5V -> Net-(C3-Pad2)
- C5 pad 1: GND -> V5
- C5 pad 2: +3.3V -> GND
- E1 pad 1: Net-(E1-antenna) -> Net-(C3-Pad2)
- J1 pad SH1: unconnected-(J1-SHIELD-PadSH1) -> GND
- J1 pad SH2: unconnected-(J1-SHIELD__1-PadSH2) -> GND
- J1 pad SH3: unconnected-(J1-SHIELD__2-PadSH3) -> GND
- J1 pad SH4: unconnected-(J1-SHIELD__3-PadSH4) -> GND
- U1 pad 5: Net-(E1-antenna) -> ANTENNA
- U1 pad 8: unconnected-(U1-V5-Pad8) -> V5
Routing:
- net +3.3V: track 0.00 -> 17.9 mm
- net +5V: track 0.00 -> 16.6 mm
- net Net-(J1-CC1_B): track 0.00 -> 10.00 mm, vias 0 -> 2
- net Net-(R3-Pad1): track 0.00 -> 9.25 mm, vias 1 -> 0
- net Net-(J1-CC1_A): track 0.00 -> 7.04 mm, vias 0 -> 2
- net PA1: track 10.3 -> 3.52 mm, vias 1 -> 0
- net GND: track 0.00 -> 5.67 mm, vias 2 -> 27
- net Net-(U1-XO): track 0.00 -> 4.28 mm
- net Net-(U1-XI): track 0.00 -> 2.43 mm
- net V5: track 0.00 -> 1.71 mm

Commit message: nearly done
Parts:
- moved J2 204.1 mm to (167.4, 121.3)
- moved C3 11.3 mm to (158.8, 129.3), turned to 90 degrees
- moved L1 9.65 mm to (155.6, 128.4)
- moved E1 6.98 mm to (152.1, 122.6), turned to 90 degrees
- moved Y1 5.85 mm to (164.3, 136.9)
- moved U1 0.75 mm to (160.3, 134.3)
Connections:
- C3 pad 2: Net-(C3-Pad2) -> ANTENNA
- E1 pad 1: Net-(C3-Pad2) -> Net-(E1-Pad1)
- J2 pad 1: unconnected-(J2-Pin_1-Pad1) -> GND
- J2 pad 2: unconnected-(J2-Pin_2-Pad2) -> +3.3V
- J2 pad 3: unconnected-(J2-Pin_3-Pad3) -> +5V
- J2 pad 4: unconnected-(J2-Pin_4-Pad4) -> PA3
- J2 pad 5: unconnected-(J2-Pin_5-Pad5) -> PA2
- J2 pad 6: unconnected-(J2-Pin_6-Pad6) -> PA7
- J2 pad 7: unconnected-(J2-Pin_7-Pad7) -> PA4
- L1 pad 1: Net-(C3-Pad2) -> Net-(E1-Pad1)
- U1 pad 1: unconnected-(U1-PA3/T/R1/SCL2/SCK_/PWM3/CP0-Pad1) -> PA3
- U1 pad 13: unconnected-(U1-PA4/SCS/PWM4/TMR2-Pad13) -> PA4
- U1 pad 16: unconnected-(U1-PA7/MOSI/T4/PWM1/TMR/RST_/CP1-Pad16) -> PA7
- U1 pad 20: unconnected-(U1-PA2/R/T1/SDA2/SCS_/PWM2/TMR1/CN-Pad20) -> PA2
Routing:
- net +3.3V: track 17.9 -> 62.6 mm
- net +5V: track 16.6 -> 46.1 mm
- net ANTENNA: track 0.00 -> 7.93 mm
- net Net-(U1-XI): track 2.43 -> 8.86 mm, vias 0 -> 2
- net PA3: track 0.00 -> 6.06 mm
- net PA4: track 0.00 -> 6.02 mm
- net GND: track 5.67 -> 0.07 mm, vias 27 -> 15
- net PA0: track 2.56 -> 8.16 mm, vias 0 -> 2
- net Net-(E1-Pad1): track 0.00 -> 5.27 mm
- net PA2: track 0.00 -> 4.16 mm
- net PA7: track 0.00 -> 3.77 mm
- net Net-(U1-XO): track 4.28 -> 7.94 mm, vias 0 -> 2
- net PA1: track 3.52 -> 6.42 mm

Commit message: big it done
its done
Parts:
- moved E1 7.65 mm to (159.7, 122.4)
- moved L1 4.49 mm to (159.7, 126.7), turned to -90 degrees
- moved C3 1.79 mm to (160.6, 128.9), turned to 180 degrees
Routing:
- net ANTENNA: track 7.93 -> 0.82 mm
- net Net-(E1-Pad1): track 5.27 -> 0.00 mm
- net GND: vias 15 -> 60
Other:
- board outline added: 16.4 x 26.4 mm

Commit message: fabrication output and fixed 5v
Parts:
- C1: value 1uF -> 0.1uF
- U2: value MIC5504-3.3YM5-TR -> the really cheap one (200mah)
- moved C2 0.21 mm to (159.0, 136.2)
Connections:
- C5 pad 1: V5 -> +5V
- U1 pad 8: V5 -> +5V
Routing:
- net +5V: track 46.0 -> 53.8 mm
- net V5: track 1.58 -> 0.00 mm

Commit message: redid and reordered
Parts:
- removed C3: 1.5pF, Personal:0603
- removed L1: 3.9nH, Personal:0603
- C1, C2, C5, C6, C7, R1, R2, R3: footprint Personal:0603 -> Footprint:0603
- E1: footprint Personal:ceramic antenna -> Footprint:DM00024648
- J1: footprint usbcport:usbcport -> Footprint:usbc
- J2: footprint fab:PinHeader_1x07_P2.54mm_Vertical_THT_D1mm -> Footprint:PinHeader_01x07_P2.54mm_Vertical_THT_D1mm
- S1: footprint Personal:button -> Footprint:button
- U1: footprint Ch572D:CH572D -> Footprint:CH572D
- U2: footprint 300mah 3.3v vreg:SOT-23-5_MC_MCH -> Footprint:voltage regulator
- Y1: footprint Personal:32mhz crystal -> Footprint:32mhz crystal
- moved E1 4.72 mm to (159.9, 127.1), turned to 0 degrees
- moved S1 0.92 mm to (167.3, 142.2)
- moved J2 0.91 mm to (167.4, 122.2)
Connections:
- E1 pad 1: Net-(E1-Pad1) -> Net-(U1-ANT)
- U1 pad 5: ANTENNA -> Net-(U1-ANT)
Routing:
- net Net-(U1-ANT): track 0.00 -> 5.56 mm
- net +5V: track 53.8 -> 54.8 mm
- net PA3: track 6.06 -> 5.22 mm
- net ANTENNA: track 0.82 -> 0.00 mm
- net Net-(R3-Pad1): track 9.25 -> 9.86 mm
- net +3.3V: track 62.6 -> 62.1 mm
- net GND: track 0.07 -> 0.45 mm, vias 60 -> 35
Other:
- board size 16.4 x 26.4 mm -> 16.4 x 25.9 mm
