File: CH572D-Board/CH572D-Board.kicad_sch (KiCad schematic)
At the start: 14 parts, among them J1 12402012E212A, U2 MIC5504-3.3YM5-TR, Y1 32mhz

Commit message: some work
Parts:
- removed C4: 0.1uF, Personal:0603, symbol 0603:C_0603
- removed E1: ~, Personal:antenna, symbol antenna:antenna
- added C6: 2.2uF, Personal:0603, symbol 0603:C_0603
- added C7: 0.1uF, Personal:0603, symbol 0603:C_0603
- added E1: AMCA31-2R450G-S1F-T3, Personal:ceramic antenna, symbol ceramic antenna:AMCA31-2R450G-S1F-T3
- added J2: Conn_PinHeader_1x07_P2.54mm_Vertical_THT_D1mm, fab:PinHeader_1x07_P2.54mm_Vertical_THT_D1mm, symbol fab:Conn_PinHeader_1x07_P2.54mm_Vertical_THT_D1mm
- added L1: 3.9nH, Personal:0603, symbol 0603:L_0603
- C3: value 10uF -> 1.5pF
- C5: value 10uF -> 2.2uF
Connections:
- net +3.3V: now also C6.1, C7.1; no longer C5.2
- net +5V: no longer C3.2
- net GND: now also C5.2, J1.SH1 (SHIELD), J1.SH2 (SHIELD__1), J1.SH3 (SHIELD__2), J1.SH4 (SHIELD__3), C6.2, C7.2; no longer C5.1
- net ANTENNA: now reaches U1.5 (ANT)
- net ANTENNA: now also L1.2
- net V5: now reaches U1.8 (V5)
- net V5: now also C5.1
- net D+ renamed PA1
- net D- renamed PA0
- new net: C3.2, E1.1, L1.1
- no-connect marks 7 -> 3
Other:
- moved on the sheet: C1, Y1

Commit message: nearly done
Connections:
- net +3.3V: now also J2.2 (Pin_2)
- net +5V: now also J2.3 (Pin_3)
- net ANTENNA: now also C3.2
- net GND: now also J2.1 (Pin_1)
- net at E1.1, L1.1: no longer C3.2
- net PA3: now reaches U1.1 (PA3/T/R1/SCL2/SCK_/PWM3/CP0)
- net PA3: now also J2.4 (Pin_4)
- net PA4: now reaches U1.13 (PA4/SCS/PWM4/TMR2)
- net PA4: now also J2.7 (Pin_7)
- net PA7: now reaches U1.16 (PA7/MOSI/T4/PWM1/TMR/RST_/CP1)
- net PA7: now also J2.6 (Pin_6)
- net PA2: now reaches U1.20 (PA2/R/T1/SDA2/SCS_/PWM2/TMR1/CN)
- net PA2: now also J2.5 (Pin_5)
Other:
- moved on the sheet: C3, E1

Commit message: big it done
its done
Parts:
- C1: value 1uF -> 0.1uF
- U2: value MIC5504-3.3YM5-TR -> the really cheap one (200mah)
Changed lines of the file:
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@@
 		(on_board yes)
 		(dnp no)
-		(fields_autoplaced yes)
 		(property "Reference" "C1"
-			(at 196.215 39.3699 90)
+			(at 196.85 39.3699 90)
 			(effects
 				(font
@@
 			)
 		)
-		(property "Value" "1uF"
-			(at 196.215 41.9099 90)
+		(property "Value" "0.1uF"
+			(at 194.31 43.815 90)
 			(effects
 				(font
@@
 			)
 		)
-		(property "Value" "MIC5504-3.3YM5-TR"
+		(property "Value" "the really cheap one (200mah)"
 			(at 220.345 27.94 0)
 			(effects

Commit message: fabrication output and fixed 5v
Connections:
- net V5 is gone; now on net +5V: C5.1, U1.8 (V5)
Other:
- moved on the sheet: C5, U1

Commit message: redid and reordered
Parts:
- removed C3: 1.5pF, Personal:0603, symbol 0603:C_0603
- removed L1: 3.9nH, Personal:0603, symbol 0603:L_0603
- C1, C2, C5, C6, C7, R1, R2, R3: footprint Personal:0603 -> Footprint:0603
- E1: footprint Personal:ceramic antenna -> Footprint:DM00024648
- J1: footprint usbcport:usbcport -> Footprint:usbc
- J2: footprint fab:PinHeader_1x07_P2.54mm_Vertical_THT_D1mm -> Footprint:PinHeader_01x07_P2.54mm_Vertical_THT_D1mm
- S1: footprint Personal:button -> Footprint:button
- U1: footprint Ch572D:CH572D -> Footprint:CH572D
- U2: footprint 300mah 3.3v vreg:SOT-23-5_MC_MCH -> Footprint:voltage regulator
- Y1: footprint Personal:32mhz crystal -> Footprint:32mhz crystal
Connections:
- net ANTENNA is gone; now on an unnamed net: U1.5 (ANT)
Other:
- moved on the sheet: E1
